File: hardware/kicad/drone_board/neurofly_drone.kicad_sch (KiCad schematic)
At the start: 0 parts

Commit message: feat: complete interactive drone deep-dive explorer with PID simulation, Autopilot Demo mode, comprehensive curriculum, and unified branding
Other:
- company: Hisar IdeaLab / FabLab Network -> Hisar IdeaLab FabLab (MIT Edgerton Center Hub)
Changed lines of the file:
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@@
     (date "2026-10-22")
     (rev "v1.0")
-    (company "Hisar IdeaLab / FabLab Network")
+    (company "Hisar IdeaLab FabLab (MIT Edgerton Center Hub)")
     (comment 1 "Seeed Studio XIAO ESP32-C6 Carrier Board")
     (comment 2 "4x Coreless Brushed Motor Driver with Flyback Diodes")
